Commit message: Add ros controller config

File: launch/test.urdf (robot description, URDF)
Before this commit: robot example, 5 links, 4 joints
Joints:
- removed joint test_joint1
- removed joint test_joint2
- removed joint test_joint3
- removed joint test_joint4
- added joint backward_left_joint: type continuous, parent base, child link3
- added joint backward_right_joint: type continuous, parent base, child link4
- added joint forward_left_joint: type continuous, parent base, child link1
- added joint forward_right_joint: type continuous, parent base, child link2
